File: node/magfield-node.kicad_sch (KiCad schematic)
At the start: 22 parts, among them J1 UPDI-PADS, J2 S4B-PH-SM4-TB, Q1 FS8205A, SW1 MSK12C02-class SPDT, U1 ATtiny1616-MNR, U2 BMM150, U3 DW01A, U4 XC6206P302MR

Commit message: Standardize node parts to LCSC/JLCPCB-PCBA verified BOM; fix CPL coordinates
Parts:
- BT1: MPN (none) -> MY-2032-10
- C1, C2, C6, C7: LCSC (none) -> C1591; MPN (none) -> CL10B104KB8NNNC
- C3: LCSC (none) -> C19702; MPN (none) -> CL10A106KP8NNNC
- C4, C5: LCSC (none) -> C15849; MPN (none) -> CL10A105KB8NNNC
- D1: MPN (none) -> WS2812B-MINI-V3/W
- J2: MPN (none) -> S4B-PH-SM4-TB(LF)(SN)
- Q1: MPN (none) -> FS8205A
- R1: LCSC (none) -> C22775; MPN (none) -> 0603WAF1000T5E
- R2: LCSC (none) -> C21190; MPN (none) -> 0603WAF1001T5E
- R3: LCSC (none) -> C23025; MPN (none) -> 0603WAF3000T5E
- R4, R5: LCSC (none) -> C23162; MPN (none) -> 0603WAF4701T5E
- SW1: value MSK12C02-class SPDT -> MSK12C02; LCSC (none) -> C431540; MPN (none) -> MSK12C02
- U1: MPN (none) -> ATTINY1616-MNR
- U2: MPN (none) -> BMM150
- U3: MPN (none) -> DW01A
- U4: value XC6206P302MR -> XC6206P302MR-G; LCSC (none) -> C9972; MPN (none) -> XC6206P302MR-G
