File: node/magfield-node.kicad_pcb (KiCad board)
At the start: 2 copper layers, 32 x 32 mm, 22 parts, among them J1 UPDI-PADS, J2 S4B-PH-SM4-TB, Q1 FS8205A, SW1 MSK12C02-class SPDT, U1 ATtiny1616-MNR, U2 BMM150, U3 DW01A, U4 XC6206P302MR

Commit message: Node: add M2 mounting holes (NW-SE); add charge hub schematic, DESIGN, BOM/CPL and READMEs
Parts:
- added MH1: MountingHole_2.2mm_M2, MountingHole_2.2mm_M2, F.Cu at (3.15, 3.60)
- added MH2: MountingHole_2.2mm_M2, MountingHole_2.2mm_M2, F.Cu at (29.3, 29.3)
- moved J1 10.9 mm to (5.00, 15.6), turned to 90 degrees
Routing:
- net SDA: track 42.5 -> 33.4 mm, vias 2 -> 4
- net UPDI: track 47.3 -> 53.4 mm, vias 3 -> 4
- net VBAT: track 81.3 -> 82.8 mm
- net GND: track 39.8 -> 39.0 mm
